File: UNY-RS-RAT-001-PCB-01 Recovery Actuation and Tracking/UNY-RS-RAT-001-PCB-01/schematics/CPU_package.kicad_sch (KiCad schematic)
At the start: 20 parts, among them J6 Conn_ST_STDC14, U15 W25Q128JVS, U2 STM32G474RETx, Y1 ECS-3225MV-240-CN-TR

Commit message: Semi complete, missing footprints and connectors
Parts:
- added R55: 10kR, Resistor_SMD:R_0603_1608Metric, symbol Device:R
Connections:
- net Psense_CS: now reaches U2.24 (PB0)
- net at U2.4 (PC15): now also R55.1
- net Fsense_CS: now reaches U2.51 (PA15)
- net Fsense_SCK: now reaches U2.56 (PB3)
- net Fsense_SDO: now reaches U2.57 (PB4)
- net Fsense_SDI: now reaches U2.58 (PB5)
- new net Received_Feedback: R55.2
- no-connect marks 4 -> 37
Other:
- note added: "SPI Connections"
- company: (none) -> E.R.I.G. e.V
