File: UNY-RS-RAT-001-PCB-01 Recovery Actuation and Tracking/UNY-RS-RAT-001-PCB-01/schematics/UNY-RS-RAT-001-PLN-00.kicad_sch (KiCad schematic)
At the start: 0 parts

Commit message: First draft for ERBUS, Power & CPU
Other:
- title: RAT High level schematics -> Sensor MCU
Changed lines of the file:
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@@
 	(paper "A4")
 	(title_block
-		(title "RAT High level schematics")
+		(title "Sensor MCU")
 		(date "2025-08-23")
 		(rev "0")

Commit message: Semi complete, missing footprints and connectors
Other:
- company: E.R.I.G. e.V. -> E.R.I.G. e.V
Changed lines of the file:
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@@
 		(date "2025-08-23")
 		(rev "0")
-		(company "E.R.I.G. e.V.")
+		(company "E.R.I.G. e.V")
 	)
 	(text "Principle Assembly and Routing Diagram"
