File: UNY-RS-RAT-001-PCB-01 Recovery Actuation and Tracking/UNY-RS-RAT-001-PCB-01/schematics/controller_unit.kicad_sch (KiCad schematic)
At the start: 0 parts

Commit message: First draft for ERBUS, Power & CPU
Other:
- added sheet Deployment Controller (light_CPU_package.kicad_sch)
- added sheet Sensor Controller (CPU_package.kicad_sch)
- title: RAT High level schematics -> Sensor MCU

Commit message: Semi complete, missing footprints and connectors
Other:
- sheet Deployment Controller ports: added {ERBUS_SIG}; removed ARM_check, MP0_IN, MP1_IN, MP2_IN, MP3_IN, MP4_IN, MP5_IN, MP6_IN, MP7_IN
- sheet Sensor Controller ports: added Received_Feedback, {CAN2_INT}, {SPI_Fsense}, {SPI_Psense}; removed none
- company: (none) -> E.R.I.G. e.V
- title: Sensor MCU -> Controller Units
