File: UNY-RS-RAT-001-PCB-01 Recovery Actuation and Tracking/UNY-RS-RAT-001-PCB-01/schematics/feedback_input.kicad_sch (KiCad schematic)
At the start: 0 parts

Commit message: First draft for ERBUS, Power & CPU
Parts:
- added C10: 100n, symbol Device:C
- added U5: HSCDANN150PASA5, RAT_foot_Library:HSCDANN150PASA5, symbol RAT_symbols:HSCDANN150PASA5
Connections:
- new net: U5.6 (NC), U5.7 (NC), U5.8 (NC)
- new net +3V3: C10.1, U5.2 (Vcc)
- new net GND: C10.2, U5.1 (P1)
- new net PRES_CS: U5.5 (P5)
- new net PRES_MISO: U5.3 (P3)
- new net PRES_SCK: U5.4 (P4)
Other:
- note added: "Pressure Sensor"
- title: RAT High level schematics -> Sensor MCU

Commit message: Semi complete, missing footprints and connectors
Parts:
- added C12, C13: 100nF, Capacitor_SMD:C_0603_1608Metric, symbol Device:C
- added FB5, FB7: 470R, Resistor_SMD:R_0603_1608Metric, symbol Device:FerriteBead
- added R39, R40, R41, R42, R43, R44: 10kR, Resistor_SMD:R_0603_1608Metric, symbol Device:R
- added R45, R46, R47, R48, R49, R50, R51, R52, R53, R54: 0, Resistor_SMD:R_0603_1608Metric, symbol Device:R
- added U7: MCP3561R, symbol RAT_symbols:MCP3561R
- added Y3: IQXO-540_831056239, Crystal_SMD_Wurth:Y_Wurth_WE-SPXO-IQXO-540, symbol Crystal_Wurth_WE-SPXO:IQXO-540_831056239
- C10: footprint (none) -> Capacitor_SMD:C_0603_1608Metric
Connections:
- net +3V3: now also FB5.2, FB7.2; no longer C10.1, U5.2 (Vcc)
- net GND: now also C12.2, C13.2, R41.2, R42.2, R44.2, U7.19 (DGND), U7.2 (AGND), U7.3 (REFIN-), Y3.2 (GND)
- net PRES_CS renamed Psense_CS
- net PRES_MISO renamed Psense_SDO
- net PRES_SCK renamed Psense_SCK
- new net: C10.1, FB5.1, U5.2 (Vcc)
- new net: R47.2, R48.1, R49.1
- new net: R40.2, R42.1, R52.2
- new net: R43.2, R44.1, R50.2
- new net: R41.1, R45.2, R46.1, R51.1
- new net: R39.2, U7.17 (IRQ/MDAT)
- new net: U7.18 (MCLK), Y3.3 (OUT)
- new net: U7.10 (NC), U7.11 (NC), U7.12 (NC), U7.7 (NC), U7.8 (NC), U7.9 (NC)
- new net 3v3_Fsense: C12.1, C13.1, FB7.1, R39.1, R40.1, R43.1, U7.1 (AVDD), U7.20 (DVDD), U7.4 (REFIN+), Y3.1 (E/D), Y3.4 (+VS)
- new net F_IN_0: R45.1, R47.1, R53.1
- new net F_IN_1: R46.2, R48.2, R54.2
- new net F_sense_CH0: R49.2, R51.2, R53.2, U7.5 (CH0)
- new net F_sense_CH1: R50.1, R52.1, R54.1, U7.6 (CH1)
- new net Fsense_CS: U7.13 (CS)
- new net Fsense_SCK: U7.14 (SCK)
- new net Fsense_SDI: U7.15 (SDI)
- new net Fsense_SDO: U7.16 (SDO)
Other:
- note added: "1/2 bridge"
- note added: "1/4 bridge"
- note added: "Connector"
- note added: "DMS amplifier & ADC"
- note added: "full bridge"
- company: (none) -> E.R.I.G. e.V
- moved on the sheet: C10, U5
