File: UNY-RS-RAT-001-PCB-01 Recovery Actuation and Tracking/UNY-RS-RAT-001-PCB-01/schematics/light_CPU_package.kicad_sch (KiCad schematic)
At the start: 42 parts, among them J1 Conn_ST_STDC14, U3 STM32G474RETx, Y2 ECS-3225MV-240-CN-TR

Commit message: Semi complete, missing footprints and connectors
Parts:
- R10, R16, R19, R22, R25, R28, R32, R35, R38: now not fitted
Other:
- company: (none) -> E.R.I.G. e.V
- title: Sensor MCU -> Deployment MCU
- moved on the sheet: R36, R37
