File: UNY-RS-RAT-001-PCB-01 Recovery Actuation and Tracking/UNY-RS-RAT-001-PCB-01/schematics/main_can.kicad_sch (KiCad schematic)
At the start: 12 parts, among them U4 SN65HVD230DR

Commit message: Semi complete, missing footprints and connectors
Other:
- title: Sensor MCU -> CAN Transciever
Changed lines of the file:
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@@
 	(paper "A4")
 	(title_block
-		(title "Sensor MCU")
+		(title "CAN Transciever")
 		(date "2025-08-23")
 		(rev "0")
@@
 		(at 157.48 88.9)
 	)
+	(bus_entry
+		(at 49.53 90.17)
+		(size -2.54 -2.54)
+		(stroke
+			(width 0)
+			(type default)
+		)
+	)
+	(bus_entry
+		(at 57.15 90.17)
+		(size -2.54 -2.54)
+		(stroke
+			(width 0)
+			(type default)
+		)
+	)
 	(wire
 		(pts
@@
 		)
 	)
+	(bus
+		(pts
+			(xy 54.61 87.63) (xy 46.99 87.63)
+		)
+		(stroke
+			(width 0)
+			(type default)
+		)
+	)
 	(wire
 		(pts
@@
 	(wire
 		(pts
+			(xy 49.53 91.44) (xy 49.53 90.17)
+		)
+		(stroke
+			(width 0)
+			(type default)
+		)
+	)
+	(wire
+		(pts
 			(xy 101.6 93.98) (xy 85.09 93.98)
 		)
@@
 		)
 	)
+	(bus
+		(pts
+			(xy 46.99 87.63) (xy 41.91 87.63)
+		)
+		(stroke
+			(width 0)
+			(type default)
+		)
+	)
 	(wire
 		(pts
@@
 	(wire
 		(pts
+			(xy 57.15 91.44) (xy 57.15 90.17)
+		)
+		(stroke
+			(width 0)
+			(type default)
+		)
+	)
+	(wire
+		(pts
 			(xy 217.17 109.22) (xy 217.17 113.03)
 		)
@@
 			(width 0)
 			(type default)
+		)
+	)
+	(label "CAN2_TX"
+		(at 49.53 91.44 270)
+		(effects
+			(font
+				(size 1.27 1.27)
+				(bold yes)
+			)
+			(justify right bottom)
 		)
 	)
@@
 			)
 			(justify left bottom)
+		)
+	)
+	(label "CAN2_RX"
+		(at 57.15 91.44 270)
+		(effects
+			(font
+				(size 1.27 1.27)
+				(bold yes)
+			)
+			(justify right bottom)
 		)
 	)
@@
 		)
 	)
-	(hierarchical_label "{CAN2_INT}"
-		(shape bidirectional)
-		(at 39.37 100.33 270)
-		(effects
-			(font
-				(size 1.27 1.27)
-				(bold yes)
-			)
-			(justify right)
-		)
-	)
 	(hierarchical_label "CANL"
 		(shape bidirectional)
@@
 		)
 	)
+	(hierarchical_label "{CAN2_INT}"
+		(shape bidirectional)
+		(at 41.91 87.63 180)
+		(effects
+			(font
+				(size 1.27 1.27)
+				(bold yes)
+			)
+			(justify right)
+		)
+	)
